File: Wireless Sensor Packet/WSPPCB/Wireless Sensor Packet/WSP2.brd (EAGLE design)
At the start: 160 x 100 mm, 58 parts, among them Q1 8/16/20MHz, U1 MCP73831, U2 MIC5205, U3 ATMEGA328, U4 MPU-9150, X1 Micro USB

Commit message: WSPPCB Update
Created initial component layout for PCB
Parts:
- removed D1, D2: U57X32, led:U57X32
- removed JP10, JP11, JP18, JP19: FIDUCIALUFIDUCIAL, SparkFun:MICRO-FIDUCIAL
- removed JP16: LOGO-SFENW2, SparkFun-Aesthetics:SFE-NEW-WEB
- removed JP17: LOGO-SFESK, SparkFun-Aesthetics:SFE-LOGO-FLAME
- removed JP3, JP4: FIDUCIAL1X2, SparkFun:FIDUCIAL-1X2
- removed JP9: FTDI Basic, SparkFun:1X06
- removed LED1: Red, Testing:0603-LED-ALT1
- removed U$1: CREATIVE_COMMONS, SparkFun:CREATIVE_COMMONS
- removed U$11: LOGO-SFENEW, SparkFun:SFE-NEW-WEBLOGO
- removed U$2: LOGO-SFESK, SparkFun:SFE-LOGO-FLAME
- removed U$3: OSHW-LOGOS, SparkFun:OSHW-LOGO-S
- removed U$4: OSHW-LOGOS, SparkFun-Aesthetics:OSHW-LOGO-S
- removed U$5: TACTILE-SWITCH-PTH, GeekAmmo:TAC-SWITCH-PTH
- added ARDPWR: Red, Testing:0603-LED-ALT1
- added FLEX1, FLEX2: (no value), wirepad:1,6/0,9
- added FTDI: FTDI Basic, SparkFun:1X06
- added ISP: AVR_SPI_PRG_6PTH, SparkFun-Connectors:2X3
- added PIN3LED, PIN4LED: (no value), SparkFun-LED:LED-0603
- added PROGRESET: TACTILE-SWITCH-PTH, GeekAmmo:TAC-SWITCH-PTH
- added R10, R9: 560, resistor:M1206
- added R12: 10K, resistor:M1206
- added R13: 22K, resistor:M1206
- added RFROW1, RFROW2: (no value), SparkFun-Connectors:1X04-1.27MM
- JP1: value LOGO-SFESK -> STAND-OFF; device SparkFun:SFE-LOGO-FLAME -> SparkFun-Electromechanical:STAND-OFF
- JP2: device SparkFun:STAND-OFF -> SparkFun-Electromechanical:STAND-OFF
- moved JP14 186.7 mm to (-31.1, 19.7)
- moved JP2 156.9 mm to (18.7, 21.0)
- moved C10 149.1 mm to (9.53, 0.95), turned to 90 degrees
- moved C13 135.0 mm to (14.9, 6.03), turned to 90 degrees
- moved SJ2 134.5 mm to (19.4, 1.91)
- moved U2 133.7 mm to (17.8, 12.4), turned to 90 degrees
- moved R7 127.0 mm to (11.7, 0.95), turned to 270 degrees
- moved SJ1 118.9 mm to (15.9, -1.27)
- moved R8 111.0 mm to (13.7, 0.95), turned to 270 degrees
- moved D11 109.4 mm to (2.86, -8.89)
- moved U3 102.4 mm to (6.99, 14.0)
- moved U1 100.6 mm to (3.17, -5.40)
- moved JP1 92.6 mm to (19.1, -8.57)
- moved U4 92.1 mm to (19.7, 6.99), turned to 180 degrees
- moved R1 86.9 mm to (14.0, 11.1), turned to 270 degrees
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Connections:
- new net N$10: PIN3LED.A, R10.2
- new net N$11: PROGRESET.4, R12.1
- new net N$9: PIN4LED.A, R9.2
- net A0: now also FLEX2.1, R13.2
- net D10: now also RFROW1.3
- net D2: now also PROGRESET.3
- net D3: now also PIN3LED.C
- net D4: now also PIN4LED.C
- net D9: now also RFROW2.3
- net DTR: now also FTDI.1; no longer JP9.1
- net GND: now also FTDI.5, FTDI.6, ISP.6, R10.1, R12.2, R13.1, R9.1, RFROW2.4; no longer JP9.5, JP9.6
- net MISO: now also ISP.1, RFROW2.1
- net MOSI: now also ISP.4, RFROW1.2
- net N$4: now also ARDPWR.A; no longer LED1.A
- net N$5: now also ARDPWR.C; no longer LED1.C
- net RAW: now also ISP.2
- net RESET: now also ISP.5
- net RXI: now also FTDI.3; no longer JP9.3
- net SCK: now also ISP.3, RFROW2.2
- net TXO: now also FTDI.2; no longer JP9.2
- net VCC: now also FLEX1.1, FTDI.4, PROGRESET.1, RFROW1.4; no longer JP9.4
Other:
- board outline removed

Commit message: Rev A of WSP PCB
Parts:
- R10, R12, R13, R9: device resistor:M1206 -> SparkFun-Resistors:0603-RES
- moved D3 56.7 mm to (34.9, 40.1), turned to 90 degrees
- moved JP15 52.2 mm to (35.6, 2.54)
- moved R8 49.4 mm to (28.9, 47.9)
- moved C19 49.2 mm to (35.2, 14.0), turned to 90 degrees
- moved R12 48.7 mm to (34.9, 21.6), turned to 180 degrees
- moved C7 46.5 mm to (24.8, 47.5)
- moved SJ3** 46.0 mm to (21.1, 41.6), turned to 90 degrees
- moved R9 45.9 mm to (34.8, 18.2)
- moved RFROW1 45.3 mm to (32.8, 34.6), turned to 180 degrees
- moved SJ2** 44.8 mm to (14.9, 46.7)
- moved C9 44.7 mm to (17.5, 41.1), turned to 180 degrees
- moved R7 44.5 mm to (11.0, 45.5), turned to 0 degrees
- moved RFROW2 44.5 mm to (32.8, 32.7), turned to 180 degrees
- moved R13 44.5 mm to (20.0, 37.9), turned to 180 degrees
- moved ISP 44.4 mm to (31.4, 41.3), turned to 180 degrees
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Connections:
- new net 3.3V: FLEX1.1, FTDI.4, PROGRESET.1, RFROW1.4
- net VCC: no longer FLEX1.1, FTDI.4, PROGRESET.1, RFROW1.4
Routing:
- net VCC: track 0.00 -> 137.9 mm, vias 0 -> 4
- net RESET: track 0.00 -> 94.9 mm, vias 0 -> 3
- net GND: track 0.00 -> 77.5 mm, vias 0 -> 14
- net RAW: track 0.00 -> 74.1 mm
- net 3.3V: track 0.00 -> 53.2 mm
- net SCK: track 0.00 -> 40.8 mm, vias 0 -> 1
- net A0: track 0.00 -> 38.8 mm, vias 0 -> 2
- net D3: track 0.00 -> 37.0 mm, vias 0 -> 2
- net D4: track 0.00 -> 33.7 mm, vias 0 -> 2
- net SDA: track 0.00 -> 33.2 mm
- net MISO: track 0.00 -> 32.0 mm
- net D2: track 0.00 -> 22.5 mm, vias 0 -> 2
- net CHARGEOUT: track 0.00 -> 21.4 mm
- net A5: track 0.00 -> 20.9 mm, vias 0 -> 2
- net MOSI: track 0.00 -> 20.2 mm, vias 0 -> 1
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- added copper zone on layer 1, net GND
- added copper zone on layer 16, net GND
Other:
- board outline added: 38.4 x 50.8 mm
- board text added: "1"
- board text added: "WSP REV A"
