File: Wireless Sensor Packet/WSPPCB/Wireless Sensor Packet/WSP2.sch (EAGLE design)
At the start: 46 parts, among them Q1 8/16/20MHz, U1 MCP73831, U2 MIC5205, U3 ATMEGA328, U4 MPU-9150, X1 Micro USB

Commit message: WSPPCB Update
Created initial component layout for PCB
Parts:
- removed D1, D2: U57X32, led:U57X32
- removed JP1: LOGO-SFESK, SparkFun:LOGO-SFESK
- removed JP2: STAND-OFF, SparkFun:STAND-OFF
- removed JP3, JP4: FIDUCIAL1X2, SparkFun:FIDUCIAL1X2
- removed JP9: FTDI Basic, SparkFun:ARDUINO_SERIAL_PROGRAMPTH
- removed U$1: CREATIVE_COMMONS, SparkFun:CREATIVE_COMMONS
- added FLEX1, FLEX2: (no value), wirepad:1,6/0,9
- added FTDI: FTDI Basic, SparkFun:ARDUINO_SERIAL_PROGRAMPTH
- added ISP: AVR_SPI_PRG_6PTH, SparkFun-Connectors:AVR_SPI_PRG_6PTH
- added PIN3LED, PIN4LED: (no value), SparkFun-LED:LED0603
- added R10, R9: 560, resistor:R-US_M1206
- added R12: 10K, resistor:R-US_M1206
- added R13: 22K, resistor:R-US_M1206
- added RFROW1, RFROW2: (no value), SparkFun-Connectors:M041.27MM
- renumbered LED1 to ARDPWR, U$5 to PROGRESET
Connections:
- new net N$10: PIN3LED.A, R10.2
- new net N$11: PROGRESET.4, R12.1
- new net N$9: PIN4LED.A, R9.2
- net A0: now also FLEX2.P, R13.2
- net D10: now also RFROW1.3
- net D2: now also PROGRESET.3
- net D3: now also PIN3LED.C
- net D4: now also PIN4LED.C
- net D9: now also RFROW2.3
- net DTR: now also FTDI.DTR; no longer JP9.DTR
- net GND: now also FTDI.CTS, FTDI.GND, ISP.6, R10.1, R12.2, R13.1, R9.1, RFROW2.4; no longer JP9.CTS, JP9.GND
- net MISO: now also ISP.1, RFROW2.1
- net MOSI: now also ISP.4, RFROW1.2
- net RAW: now also ISP.2
- net RESET: now also ISP.5
- net RXI: now also FTDI.TXO; no longer JP9.TXO
- net SCK: now also ISP.3, RFROW2.2
- net TXO: now also FTDI.RXI; no longer JP9.RXI
- net VCC: now also FLEX1.P, FTDI.VCC, PROGRESET.1, RFROW1.4; no longer JP9.VCC

Commit message: Rev A of WSP PCB
Parts:
- R10, R12, R13, R9: device resistor:R-US_M1206 -> SparkFun-Resistors:RESISTOR0603-RES
Connections:
- new net 3.3V: FLEX1.P, FTDI.VCC, PROGRESET.1, RFROW1.4
- net VCC: no longer FLEX1.P, FTDI.VCC, PROGRESET.1, RFROW1.4
Changed lines of the file:
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@@
 <layer number="223" name="223bmp" color="24" fill="1" visible="no" active="no"/>
 <layer number="224" name="224bmp" color="25" fill="1" visible="no" active="no"/>
+<layer number="225" name="225bmp" color="7" fill="1" visible="yes" active="yes"/>
+<layer number="226" name="226bmp" color="7" fill="1" visible="yes" active="yes"/>
+<layer number="227" name="227bmp" color="7" fill="1" visible="yes" active="yes"/>
+<layer number="228" name="228bmp" color="7" fill="1" visible="yes" active="yes"/>
+<layer number="229" name="229bmp" color="7" fill="1" visible="yes" active="yes"/>
+<layer number="230" name="230bmp" color="7" fill="1" visible="yes" active="yes"/>
+<layer number="231" name="231bmp" color="7" fill="1" visible="yes" active="yes"/>
 <layer number="248" name="Housing" color="7" fill="1" visible="yes" active="yes"/>
 <layer number="249" name="Edge" color="7" fill="1" visible="yes" active="yes"/>
@@
 <part name="FLEX1" library="wirepad" deviceset="1,6/0,9" device=""/>
 <part name="FLEX2" library="wirepad" deviceset="1,6/0,9" device=""/>
-<part name="R13" library="resistor" deviceset="R-US_" device="M1206" value="22K"/>
-<part name="R9" library="resistor" deviceset="R-US_" device="M1206" value="560"/>
-<part name="R10" library="resistor" deviceset="R-US_" device="M1206" value="560"/>
+<part name="R13" library="SparkFun-Resistors" deviceset="RESISTOR" device="0603-RES" value="22K"/>
+<part name="R9" library="SparkFun-Resistors" deviceset="RESISTOR" device="0603-RES" value="560"/>
+<part name="R10" library="SparkFun-Resistors" deviceset="RESISTOR" device="0603-RES" value="560"/>
 <part name="GND13" library="SparkFun-Aesthetics" deviceset="GND" device=""/>
 <part name="GND22" library="SparkFun-Aesthetics" deviceset="GND" device=""/>
 <part name="GND23" library="supply1" deviceset="GND" device=""/>
-<part name="R12" library="resistor" deviceset="R-US_" device="M1206" value="10K"/>
+<part name="R12" library="SparkFun-Resistors" deviceset="RESISTOR" device="0603-RES" value="10K"/>
 <part name="GND24" library="SparkFun-Aesthetics" deviceset="GND" device=""/>
 <part name="RFROW1" library="SparkFun-Connectors" deviceset="M04" device="1.27MM"/>
 <part name="RFROW2" library="SparkFun-Connectors" deviceset="M04" device="1.27MM"/>
+<part name="GND27" library="SparkFun" deviceset="GND" device=""/>
+<part name="GND29" library="SparkFun" deviceset="GND" device=""/>
+<part name="P+9" library="SparkFun" deviceset="3.3V" device="" value="VCC"/>
+<part name="P+10" library="SparkFun" deviceset="3.3V" device="" value="VCC"/>
+<part name="GND31" library="SparkFun" deviceset="GND" device=""/>
+<part name="P+12" library="SparkFun" deviceset="3.3V" device="" value="VCC"/>
+<part name="P+13" library="SparkFun" deviceset="3.3V" device="" value="VCC"/>
 </parts>
 <sheets>
@@
 <instance part="RFROW1" gate="G$1" x="68.58" y="104.14"/>
 <instance part="RFROW2" gate="G$1" x="104.14" y="104.14"/>
+<instance part="GND27" gate="1" x="101.6" y="137.16" rot="R90"/>
+<instance part="GND29" gate="1" x="109.22" y="134.62" rot="R90"/>
+<instance part="P+9" gate="G$1" x="99.06" y="132.08" rot="R270"/>
+<instance part="P+10" gate="G$1" x="83.82" y="109.22" rot="R270"/>
+<instance part="GND31" gate="1" x="121.92" y="109.22" rot="R90"/>
+<instance part="P+12" gate="G$1" x="30.48" y="91.44" rot="R270"/>
+<instance part="P+13" gate="G$1" x="149.86" y="172.72" rot="R90"/>
 </instances>
 <busses>
@@
 </segment>
 <segment>
-<wire x1="91.44" y1="134.62" x2="93.98" y2="134.62" width="0.1524" layer="91"/>
-<pinref part="FTDI" gate="G$1" pin="CTS"/>
-<label x="93.98" y="134.62" size="1.27" layer="95" xref="yes"/>
-</segment>
-<segment>
-<wire x1="91.44" y1="137.16" x2="93.98" y2="137.16" width="0.1524" layer="91"/>
-<pinref part="FTDI" gate="G$1" pin="GND"/>
-<label x="93.98" y="137.16" size="1.27" layer="95" xref="yes"/>
-</segment>
-<segment>
 <pinref part="GND28" gate="1" pin="GND"/>
 <pinref part="R11" gate="G$1" pin="1"/>
@@
 </segment>
 <segment>
+<pinref part="FTDI" gate="G$1" pin="GND"/>
+<pinref part="GND27" gate="1" pin="GND"/>
+<wire x1="91.44" y1="137.16" x2="99.06" y2="137.16" width="0.1524" layer="91"/>
+</segment>
+<segment>
+<pinref part="FTDI" gate="G$1" pin="CTS"/>
+<pinref part="GND29" gate="1" pin="GND"/>
+<wire x1="91.44" y1="134.62" x2="106.68" y2="134.62" width="0.1524" layer="91"/>
+</segment>
+<segment>
 <pinref part="RFROW2" gate="G$1" pin="4"/>
-<wire x1="109.22" y1="109.22" x2="111.76" y2="109.22" width="0.1524" layer="91"/>
-<label x="111.76" y="109.22" size="1.778" layer="95" xref="yes"/>
+<pinref part="GND31" gate="1" pin="GND"/>
+<wire x1="109.22" y1="109.22" x2="119.38" y2="109.22" width="0.1524" layer="91"/>
 </segment>
 </net>
@@
 </segment>
 <segment>
-<wire x1="91.44" y1="132.08" x2="93.98" y2="132.08" width="0.1524" layer="91"/>
-<pinref part="FTDI" gate="G$1" pin="VCC"/>
-<label x="93.98" y="132.08" size="1.27" layer="95" xref="yes"/>
-</segment>
-<segment>
 <wire x1="223.52" y1="157.48" x2="223.52" y2="160.02" width="0.1524" layer="91"/>
 <pinref part="P+2" gate="G$1" pin="3.3V"/>
@@
 <junction x="83.82" y="162.56"/>
 </segment>
-<segment>
-<pinref part="FLEX1" gate="1" pin="P"/>
-<wire x1="25.4" y1="91.44" x2="30.48" y2="91.44" width="0.1524" layer="91"/>
-<label x="30.48" y="91.44" size="1.778" layer="95" xref="yes"/>
-</segment>
-<segment>
-<pinref part="PROGRESET" gate="G$1" pin="1"/>
-<wire x1="160.02" y1="172.72" x2="157.48" y2="172.72" width="0.1524" layer="91"/>
-<label x="157.48" y="172.72" size="1.778" layer="95" rot="R180" xref="yes"/>
-</segment>
-<segment>
-<pinref part="RFROW1" gate="G$1" pin="4"/>
-<wire x1="73.66" y1="109.22" x2="78.74" y2="109.22" width="0.1524" layer="91"/>
-<label x="78.74" y="109.22" size="1.778" layer="95" xref="yes"/>
-</segment>
 </net>
 <net name="RAW" class="1">
@@
 </segment>
 </net>
+<net name="3.3V" class="0">
+<segment>
+<pinref part="FTDI" gate="G$1" pin="VCC"/>
+<pinref part="P+9" gate="G$1" pin="3.3V"/>
+<wire x1="91.44" y1="132.08" x2="99.06" y2="132.08" width="0.1524" layer="91"/>
+</segment>
+<segment>
+<pinref part="RFROW1" gate="G$1" pin="4"/>
+<pinref part="P+10" gate="G$1" pin="3.3V"/>
+<wire x1="73.66" y1="109.22" x2="83.82" y2="109.22" width="0.1524" layer="91"/>
+</segment>
+<segment>
+<pinref part="FLEX1" gate="1" pin="P"/>
+<pinref part="P+12" gate="G$1" pin="3.3V"/>
+<wire x1="25.4" y1="91.44" x2="30.48" y2="91.44" width="0.1524" layer="91"/>
+</segment>
+<segment>
+<pinref part="PROGRESET" gate="G$1" pin="1"/>
+<pinref part="P+13" gate="G$1" pin="3.3V"/>
+<wire x1="160.02" y1="172.72" x2="149.86" y2="172.72" width="0.1524" layer="91"/>
+</segment>
+</net>
